Commit message: Updates Macaroni model to match current physical car.

File: rr_description/urdf/macaroni.urdf (robot description, URDF)
Before this commit: robot macaroni, 14 links, 13 joints
Links:
- removed link laser
- link chassis: geometry collision mesh filename=package://rr_description/meshes/Macaroni.dae; visual mesh filename=package://rr_description/meshes/Macaroni.dae
- link wheel_back_left: geometry collision mesh filename=package://rr_description/meshes/Macaroni-wheel.dae; visual mesh filename=package://rr_description/meshes/Macaroni-wheel.dae
- link wheel_back_right: geometry collision mesh filename=package://rr_description/meshes/Macaroni-wheel.dae; visual mesh filename=package://rr_description/meshes/Macaroni-wheel.dae
- link wheel_front_left: geometry collision mesh filename=package://rr_description/meshes/Macaroni-wheel.dae; visual mesh filename=package://rr_description/meshes/Macaroni-wheel.dae
- link wheel_front_right: geometry collision mesh filename=package://rr_description/meshes/Macaroni-wheel.dae; visual mesh filename=package://rr_description/meshes/Macaroni-wheel.dae
Joints:
- removed joint lidar_joint
- joint cam_chassis_height: origin xyz=0.21793 0 0.22 rpy=0 0 0 -> xyz=0.27251 0 0.18245 rpy=0 0 0
